Commit message: added more links, sensors, cameras, etc.

File: maggie_description/robots/maggie.urdf (robot description, URDF)
Before this commit: robot maggie, 13 links, 12 joints
Links:
- added link hokuyo_link, mass 1
- added link ir_link, mass 0.02
- added link rfid_link, mass 0.02
- added link sick_link, mass 5
- added link touch_head_link, mass 0.01
- added link touch_left_back_link, mass 0.01
- added link touch_left_hand_link, mass 0.01
- added link touch_left_shoulder_link, mass 0.01
- added link touch_right_back_link, mass 0.01
- added link touch_right_hand_link, mass 0.01
- added link touch_right_shoulder_link, mass 0.01
- added link webcam_link, mass 0.03
- link left_arm_link: geometry collision box size=0.4 0.2 0.1; visual box size=0.4 0.15 0.1
- link right_arm_link: geometry collision box size=0.4 0.2 0.1; visual box size=0.4 0.15 0.1
Joints:
- added joint arm_to_touch_left_back_joint: type fixed, parent upper_base_link, child touch_left_back_link, origin xyz=-0.1 -0.18 0.15 rpy=0 0 0
- added joint arm_to_touch_left_hand_joint: type fixed, parent left_arm_link, child touch_left_hand_link, origin xyz=0.05 0 -0.4 rpy=0 0 0
- added joint arm_to_touch_left_shoulder_joint: type fixed, parent upper_base_link, child touch_left_shoulder_link, origin xyz=-0.1 0 0.25 rpy=0 0 0
- added joint arm_to_touch_right_back_joint: type fixed, parent upper_base_link, child touch_right_back_link, origin xyz=0.1 -0.18 0.15 rpy=0 0 0
- added joint arm_to_touch_right_hand_joint: type fixed, parent right_arm_link, child touch_right_hand_link, origin xyz=-0.05 0 -0.4 rpy=0 0 0
- added joint arm_to_touch_right_shoulder_joint: type fixed, parent upper_base_link, child touch_right_shoulder_link, origin xyz=0.1 0 0.25 rpy=0 0 0
- added joint base_to_hokuyo_joint: type fixed, parent base_link, child hokuyo_link, origin xyz=0 -0.2 0.2 rpy=0 0 0
- added joint base_to_ir_joint: type fixed, parent base_link, child ir_link, origin xyz=0 0.2 0.3 rpy=0 0 0
- added joint base_to_sick_joint: type fixed, parent base_link, child sick_link, origin xyz=0 0.2 0 rpy=0 0 0
- added joint head_to_rfid_joint: type fixed, parent head_link, child rfid_link, origin xyz=0 0.2 0 rpy=0 0 0
- added joint head_to_touch_head_joint: type fixed, parent head_link, child touch_head_link, origin xyz=0 0 0.2 rpy=0 0 0
- added joint mouth_to_webcam_joint: type fixed, parent mouth_link, child webcam_link, origin xyz=0 0 0 rpy=0 0 0
- joint base_to_left_arm_joint: limit lower=-1.05 upper=2.69 effort=1000.0 velocity=0.5 -> lower=-1.04716666667 upper=2.356125 effort=1000.0 velocity=0.5
- joint base_to_right_arm_joint: limit lower=-1.05 upper=2.69 effort=1000.0 velocity=0.5 -> lower=-1.04716666667 upper=2.356125 effort=1000.0 velocity=0.5

File: maggie_description/robots/maggie.urdf.xacro (robot description, xacro)
@@ -9,5 +9,5 @@
         <visual>
             <geometry>
-                <cylinder length="0.5" radius="0.2" />
+                <cylinder length="${baselen}" radius="0.2" />
             </geometry>
             <material name="white" />
@@ -15,5 +15,5 @@
         <collision>
             <geometry>
-                <cylinder length="0.5" radius="0.2" />
+                <cylinder length="${baselen}" radius="0.2" />
             </geometry>
         </collision>
@@ -23,5 +23,5 @@
         <visual>
             <geometry>
-                <cylinder length="0.5" radius="0.2" />
+                <cylinder length="${bodylen}" radius="0.2" />
             </geometry>
             <material name="blue" />
@@ -29,5 +29,5 @@
         <collision>
             <geometry>
-                <cylinder length="0.5" radius="0.2" />
+                <cylinder length="${bodylen}" radius="0.2" />
             </geometry>
         </collision>
@@ -46,5 +46,5 @@
         <origin xyz="0 0 0.45" />
         <axis xyz="0 0 1" />
-        <limit effort="1000.0" lower="-1.57075" upper="1.57075" velocity="0.5" />
+        <limit effort="1000.0" lower="-${pi/2}" upper="${pi/2}" velocity="${defaultvel}" />
     </joint>
     <link name="head_link">
@@ -67,5 +67,5 @@
         <origin xyz="0 0 0" />
         <axis xyz="1 0 0" />
-        <limit effort="1000.0" lower="-0.26" upper="0.26" velocity="0.5" />
+        <limit effort="1000.0" lower="-0.26" upper="0.26" velocity="${defaultvel}" />
     </joint>
     <!-- MOUTH -->
@@ -121,8 +121,61 @@
     <xacro:wheel prefix="left" reflect="-1" />
     <xacro:wheel prefix="right" reflect="1" />
-    <!-- SENSORS -->
+    <!-- RFID -->
+    <link name="rfid_link">
+        <xacro:default_inertial mass="0.02" />
+    </link>
+    <joint name="head_to_rfid_joint" type="fixed">
+        <parent link="head_link" />
+        <child link="rfid_link" />
+        <origin xyz="0 0.2 0" rpy="0 0 0" />
+    </joint>
+    <!-- IR CONTROLLER -->
+    <link name="ir_link">
+        <xacro:default_inertial mass="0.02" />
+    </link>
+    <joint name="base_to_ir_joint" type="fixed">
+        <parent link="base_link" />
+        <child link="ir_link" />
+        <origin xyz="0 0.2 0.3" rpy="0 0 0" />
+    </joint>
+    <!-- LASERS -->
+    <link name="sick_link">
+        <xacro:default_inertial mass="5" />
+    </link>
+    <joint name="base_to_sick_joint" type="fixed">
+        <parent link="base_link" />
+        <child link="sick_link" />
+        <origin xyz="0 0.2 0" rpy="0 0 0" />
+    </joint>
+    <link name="hokuyo_link">
+        <xacro:default_inertial mass="1" />
+    </link>
+    <joint name="base_to_hokuyo_joint" type="fixed">
+        <parent link="base_link" />
+        <child link="hokuyo_link" />
+        <origin xyz="0 -0.2 0.2" rpy="0 0 0" />
+    </joint>
+    <!-- TOUCH SENSORS -->
+    <link name="touch_head_link">
+        <xacro:default_inertial mass="0.01" />
+    </link>
+    <joint name="head_to_touch_head_joint" type="fixed">
+        <parent link="head_link" />
+        <child link="touch_head_link" />
+        <origin xyz="0 0 0.2" rpy="0 0 0" />
+    </joint>
+    <xacro:include filename="$(find maggie_description)/urdf/touch_back.urdf.xacro" />
+    <xacro:touch_back prefix="left" reflect="-1" />
+    <xacro:touch_back prefix="right" reflect="1" />
+    <xacro:include filename="$(find maggie_description)/urdf/touch_shoulders.urdf.xacro" />
+    <xacro:touch_shoulder prefix="left" reflect="-1" />
+    <xacro:touch_shoulder prefix="right" reflect="1" />
+    <xacro:include filename="$(find maggie_description)/urdf/touch_hands.urdf.xacro" />
+    <xacro:touch_hand prefix="left" reflect="-1" />
+    <xacro:touch_hand prefix="right" reflect="1" />
+    <!-- CAMERAS -->
     <link name="kinect_link">
         <visual>
-            <origin xyz="0 0 0" rpy="0 0 1.57075" />
+            <origin xyz="0 0 0" rpy="0 0 ${pi/2}" />
             <geometry>
                 <mesh filename="package://maggie_description/meshes/kinect/kinect.dae" scale="0.001 0.001 0.001" />
@@ -130,5 +183,5 @@
         </visual>
         <collision>
-            <origin xyz="0 0 0" rpy="0 0 1.57075" />
+            <origin xyz="0 0 0" rpy="0 0 ${pi/2}" />
             <geometry>
                 <mesh filename="package://maggie_description/meshes/kinect/kinect.dae" scale="0.001 0.001 0.001" />
@@ -142,3 +195,11 @@
         <origin xyz="0 0.25 0.25" rpy="0 0 0" />
     </joint>
+    <link name="webcam_link">
+        <xacro:default_inertial mass="0.03" />
+    </link>
+    <joint name="mouth_to_webcam_joint" type="fixed">
+        <parent link="mouth_link" />
+        <child link="webcam_link" />
+        <origin xyz="0 0 0" rpy="0 0 0" />
+    </joint>
 </robot>

File: maggie_description/urdf/arms.urdf.xacro (robot description, xacro)
@@ -4,14 +4,14 @@
         <link name="${prefix}_arm_link">
             <visual>
-                <origin xyz="0 0 -0.2" rpy="0 1.57075 0" />
+                <origin xyz="0 0 -0.2" rpy="0 ${pi/2} 0" />
                 <geometry>
-                    <box size="0.4 0.2 0.1" />
+                    <box size="${armlen} 0.15 0.1" />
                 </geometry>
                 <material name="white" />
             </visual>
             <collision>
-                <origin xyz="0 0 -0.2" rpy="0 1.57075 0" />
+                <origin xyz="0 0 -0.2" rpy="0 ${pi/2} 0" />
                 <geometry>
-                    <box size="0.4 0.2 0.1" />
+                    <box size="${armlen} 0.2 0.1" />
                 </geometry>
             </collision>
@@ -23,5 +23,5 @@
             <origin xyz="${reflect*0.25} 0 0.25" />
             <axis xyz="1 0 0" />
-            <limit effort="1000.0" lower="-1.05" upper="2.69" velocity="0.5" />
+            <limit effort="1000.0" lower="-${pi/3}" upper="${3*pi/4}" velocity="${defaultvel}" />
         </joint>
     </xacro:macro>

File: maggie_description/urdf/common.xacro (robot description, xacro)
@@ -5,6 +5,6 @@
     <xacro:property name="bodylen" value="0.5" />
     <xacro:property name="baselen" value="0.5" />
-    <xacro:property name="armlen" value="0.6" />
-    <xacro:property name="wheeldiam" value="0.07" />
+    <xacro:property name="armlen" value="0.4" />
+    <xacro:property name="defaultvel" value="0.5" />
     <!-- MACROS -->
     <xacro:macro name="default_inertial" params="mass">

File: maggie_description/urdf/wheels.urdf.xacro (robot description, xacro)
@@ -4,5 +4,5 @@
         <link name="${prefix}_wheel_link">
             <visual>
-                <origin xyz="0 0 0" rpy="0 0 1.57075" />
+                <origin xyz="0 0 0" rpy="0 0 ${pi/2}" />
                 <geometry>
                     <mesh filename="package://maggie_description/meshes/base/wheel.dae" />
@@ -10,5 +10,5 @@
             </visual>
             <collision>
-                <origin xyz="0 0 0" rpy="0 0 1.57075" />
+                <origin xyz="0 0 0" rpy="0 0 ${pi/2}" />
                 <geometry>
                     <mesh filename="package://maggie_description/meshes/base/wheel.dae" />

Commit message: updated parts with real meassures

File: maggie_description/robots/maggie.urdf (robot description, URDF)
Before this commit: robot maggie, 25 links, 24 joints
Links:
- added link neck_link, mass 0.2; collision cylinder length=0.05 radius=0.02; visual cylinder length=0.05 radius=0.04
- link base_link: geometry collision cylinder length=0.42 radius=0.2; visual cylinder length=0.42 radius=0.2
- link left_arm_link: geometry collision box size=0.38 0.15 0.1; visual box size=0.38 0.15 0.1
- link right_arm_link: geometry collision box size=0.38 0.15 0.1; visual box size=0.38 0.15 0.1
- link screen_link: geometry collision box size=0.16 0.02 0.21; visual box size=0.16 0.02 0.21
- link upper_base_link: geometry collision cylinder length=0.56 radius=0.2; visual cylinder length=0.56 radius=0.2
Joints:
- removed joint base_to_pan_head_joint
- added joint base_to_neck_joint: type fixed, parent upper_base_link, child neck_link, origin xyz=0 0 0.305
- added joint neck_to_pan_head_joint: type revolute, parent neck_link, child link_virtual, origin xyz=0 0 0.2, axis 0 0 1, limit lower=-1.57075 upper=1.57075 effort=1000.0 velocity=0.5
- joint arm_to_touch_left_back_joint: origin xyz=-0.1 -0.18 0.15 rpy=0 0 0 -> xyz=-0.1 -0.18 0.18 rpy=0 0 0
- joint arm_to_touch_left_hand_joint: origin xyz=0.05 0 -0.4 rpy=0 0 0 -> xyz=0.05 0 -0.36 rpy=0 0 0
- joint arm_to_touch_left_shoulder_joint: origin xyz=-0.1 0 0.25 rpy=0 0 0 -> xyz=-0.1 0 0.28 rpy=0 0 0
- joint arm_to_touch_right_back_joint: origin xyz=0.1 -0.18 0.15 rpy=0 0 0 -> xyz=0.1 -0.18 0.18 rpy=0 0 0
- joint arm_to_touch_right_hand_joint: origin xyz=-0.05 0 -0.4 rpy=0 0 0 -> xyz=-0.05 0 -0.36 rpy=0 0 0
- joint arm_to_touch_right_shoulder_joint: origin xyz=0.1 0 0.25 rpy=0 0 0 -> xyz=0.1 0 0.28 rpy=0 0 0
- joint base_to_kinect_joint: origin xyz=0 0.25 0.25 rpy=0 0 0 -> xyz=0 0.26 0.23 rpy=0 0 0
- joint base_to_left_arm_joint: origin xyz=-0.25 0 0.25 -> xyz=-0.25 0 0.28
- joint base_to_left_wheel_joint: origin xyz=-0.1 0 -0.2 rpy=0 0 0 -> xyz=-0.1 0 -0.18 rpy=0 0 0
- joint base_to_right_arm_joint: origin xyz=0.25 0 0.25 -> xyz=0.25 0 0.28
- joint base_to_right_wheel_joint: origin xyz=0.1 0 -0.2 rpy=0 0 0 -> xyz=0.1 0 -0.18 rpy=0 0 0
- joint base_to_screen_joint: origin xyz=0 0.19 0 -> xyz=0 0.19 0.105
- joint base_to_upper_base_joint: origin xyz=0 0 0.5 -> xyz=0 0 0.49

File: maggie_description/robots/maggie.urdf.xacro (robot description, xacro)
@@ -37,12 +37,32 @@
         <parent link="base_link" />
         <child link="upper_base_link" />
-        <origin xyz="0 0 0.5" />
+        <origin xyz="0 0 ${baselen/2+bodylen/2}" />
+    </joint>
+    <!-- NECK -->
+    <link name="neck_link">
+        <visual>
+            <geometry>
+                <cylinder length="0.05" radius="0.04" />
+            </geometry>
+            <material name="black" />
+        </visual>
+        <collision>
+            <geometry>
+                <cylinder length="0.05" radius="0.02" />
+            </geometry>
+        </collision>
+        <xacro:default_inertial mass="0.2" />
+    </link>
+    <joint name="base_to_neck_joint" type="fixed">
+        <parent link="upper_base_link" />
+        <child link="neck_link" />
+        <origin xyz="0 0 ${bodylen/2+0.05/2}" />
     </joint>
     <!-- HEAD -->
     <link name="link_virtual" />
-    <joint name="base_to_pan_head_joint" type="revolute">
-        <parent link="upper_base_link" />
+    <joint name="neck_to_pan_head_joint" type="revolute">
+        <parent link="neck_link" />
         <child link="link_virtual" />
-        <origin xyz="0 0 0.45" />
+        <origin xyz="0 0 ${headlen/2}" />
         <axis xyz="0 0 1" />
         <limit effort="1000.0" lower="-${pi/2}" upper="${pi/2}" velocity="${defaultvel}" />
@@ -51,5 +71,5 @@
         <visual>
             <geometry>
-                <sphere radius="0.2" />
+                <sphere radius="${headlen/2}" />
             </geometry>
             <material name="white" />
@@ -57,5 +77,5 @@
         <collision>
             <geometry>
-                <sphere radius="0.2" />
+                <sphere radius="${headlen/2}" />
             </geometry>
         </collision>
@@ -101,5 +121,5 @@
         <visual>
             <geometry>
-                <box size="0.2 0.02 0.25" />
+                <box size="0.16 0.02 0.21" />
             </geometry>
             <material name="black" />
@@ -107,5 +127,5 @@
         <collision>
             <geometry>
-                <box size="0.2 0.02 0.25" />
+                <box size="0.16 0.02 0.21" />
             </geometry>
         </collision>
@@ -115,5 +135,5 @@
         <parent link="upper_base_link" />
         <child link="screen_link" />
-        <origin xyz="0 0.19 0" />
+        <origin xyz="0 0.19 ${0.21/2}" />
     </joint>
     <!-- WHEELS -->
@@ -193,5 +213,5 @@
         <parent link="base_link" />
         <child link="kinect_link" />
-        <origin xyz="0 0.25 0.25" rpy="0 0 0" />
+        <origin xyz="0 ${baselen/2+0.05} ${baselen/2+0.02}" rpy="0 0 0" />
     </joint>
     <link name="webcam_link">

File: maggie_description/urdf/arms.urdf.xacro (robot description, xacro)
@@ -4,5 +4,5 @@
         <link name="${prefix}_arm_link">
             <visual>
-                <origin xyz="0 0 -0.2" rpy="0 ${pi/2} 0" />
+                <origin xyz="0 0 ${-armlen/2}" rpy="0 ${pi/2} 0" />
                 <geometry>
                     <box size="${armlen} 0.15 0.1" />
@@ -13,5 +13,5 @@
                 <origin xyz="0 0 -0.2" rpy="0 ${pi/2} 0" />
                 <geometry>
-                    <box size="${armlen} 0.2 0.1" />
+                    <box size="${armlen} 0.15 0.1" />
                 </geometry>
             </collision>
@@ -21,5 +21,5 @@
             <parent link="upper_base_link" />
             <child link="${prefix}_arm_link" />
-            <origin xyz="${reflect*0.25} 0 0.25" />
+            <origin xyz="${reflect*0.25} 0 ${bodylen/2}" />
             <axis xyz="1 0 0" />
             <limit effort="1000.0" lower="-${pi/3}" upper="${3*pi/4}" velocity="${defaultvel}" />

File: maggie_description/urdf/common.xacro (robot description, xacro)
@@ -3,7 +3,8 @@
     <!-- CONSTANTS -->
     <xacro:property name="pi" value="3.1415" />
-    <xacro:property name="bodylen" value="0.5" />
-    <xacro:property name="baselen" value="0.5" />
-    <xacro:property name="armlen" value="0.4" />
+    <xacro:property name="bodylen" value="0.56" />
+    <xacro:property name="baselen" value="0.42" />
+    <xacro:property name="armlen" value="0.38" />
+    <xacro:property name="headlen" value="0.4" />
     <xacro:property name="defaultvel" value="0.5" />
     <!-- MACROS -->

File: maggie_description/urdf/touch_hands.urdf.xacro (robot description, xacro)
@@ -8,5 +8,5 @@
             <parent link="${prefix}_arm_link" />
             <child link="touch_${prefix}_hand_link" />
-            <origin xyz="${reflect*-0.05} 0 -${armlen}" rpy="0 0 0" />
+            <origin xyz="${reflect*-0.05} 0 -${armlen-0.02}" rpy="0 0 0" />
         </joint>
     </xacro:macro>

File: maggie_description/urdf/wheels.urdf.xacro (robot description, xacro)
@@ -20,5 +20,5 @@
             <parent link="base_link" />
             <child link="${prefix}_wheel_link" />
-            <origin xyz="${reflect*0.1} 0 -0.2" rpy="0 0 0" />
+            <origin xyz="${reflect*0.1} 0 -0.18" rpy="0 0 0" />
             <axis xyz="1 0 0" rpy="0 0 0" />
         </joint>

Commit message: updated sick rotation

File: maggie_description/robots/maggie.urdf (robot description, URDF)
Before this commit: robot maggie, 26 links, 25 joints
Joints:
- joint base_to_sick_joint: origin xyz=0 0.2 0 rpy=0 0 0 -> xyz=0 0.2 0 rpy=1.57075 0 0

File: maggie_description/robots/maggie.urdf.xacro (robot description, xacro)
@@ -166,5 +166,5 @@
         <parent link="base_link" />
         <child link="sick_link" />
-        <origin xyz="0 0.2 0" rpy="0 0 0" />
+        <origin xyz="0 0.2 0" rpy="${pi/2} 0 0" />
     </joint>
     <link name="hokuyo_link">

Commit message: updated sick rotation

File: maggie_description/robots/maggie.urdf (robot description, URDF)
Before this commit: robot maggie, 26 links, 25 joints
Joints:
- joint base_to_sick_joint: origin xyz=0 0.2 0 rpy=1.57075 0 0 -> xyz=0 0.2 0 rpy=0 1.57075 0

File: maggie_description/robots/maggie.urdf.xacro (robot description, xacro)
@@ -166,5 +166,5 @@
         <parent link="base_link" />
         <child link="sick_link" />
-        <origin xyz="0 0.2 0" rpy="${pi/2} 0 0" />
+        <origin xyz="0 0.2 0" rpy="0 ${pi/2} 0" />
     </joint>
     <link name="hokuyo_link">

Commit message: updated sick rotation

File: maggie_description/robots/maggie.urdf (robot description, URDF)
Before this commit: robot maggie, 26 links, 25 joints
Joints:
- joint base_to_sick_joint: origin xyz=0 0.2 0 rpy=0 1.57075 0 -> xyz=0 0.2 0 rpy=0 0 1.57075

File: maggie_description/robots/maggie.urdf.xacro (robot description, xacro)
@@ -166,5 +166,5 @@
         <parent link="base_link" />
         <child link="sick_link" />
-        <origin xyz="0 0.2 0" rpy="0 ${pi/2} 0" />
+        <origin xyz="0 0.2 0" rpy="0 0 ${pi/2}" />
     </joint>
     <link name="hokuyo_link">

Commit message: updated hokuyo rotation

File: maggie_description/robots/maggie.urdf (robot description, URDF)
Before this commit: robot maggie, 26 links, 25 joints
Joints:
- joint base_to_hokuyo_joint: origin xyz=0 -0.2 0.2 rpy=0 0 0 -> xyz=0 -0.2 0.2 rpy=0 0 -1.57075

File: maggie_description/robots/maggie.urdf.xacro (robot description, xacro)
@@ -174,5 +174,5 @@
         <parent link="base_link" />
         <child link="hokuyo_link" />
-        <origin xyz="0 -0.2 0.2" rpy="0 0 0" />
+        <origin xyz="0 -0.2 0.2" rpy="0 0 -${pi/2}" />
     </joint>
     <!-- TOUCH SENSORS -->

Commit message: updated urdf and resolved bug with tf

File: maggie_description/robots/maggie.urdf (robot description, URDF)
Before this commit: robot maggie, 26 links, 25 joints
Joints:
- joint base_to_hokuyo_joint: origin xyz=0 -0.2 0.2 rpy=0 0 -1.57075 -> xyz=0 -0.2 0.46 rpy=0 0 -1.57075
- joint base_to_ir_joint: origin xyz=0 0.2 0.3 rpy=0 0 0 -> xyz=0 0.2 0.56 rpy=0 0 0
- joint base_to_kinect_joint: origin xyz=0 0.26 0.23 rpy=0 0 0 -> xyz=0 0.26 0.49 rpy=0 0 0
- joint base_to_left_wheel_joint: origin xyz=-0.1 0 -0.18 rpy=0 0 0 -> xyz=-0.1 0 0.08 rpy=0 0 0
- joint base_to_right_wheel_joint: origin xyz=0.1 0 -0.18 rpy=0 0 0 -> xyz=0.1 0 0.08 rpy=0 0 0
- joint base_to_sick_joint: origin xyz=0 0.2 0 rpy=0 0 1.57075 -> xyz=0 0.2 0.26 rpy=0 0 1.57075
- joint base_to_upper_base_joint: origin xyz=0 0 0.49 -> xyz=0 0 0.75

File: maggie_description/robots/maggie.urdf.xacro (robot description, xacro)
@@ -8,4 +8,5 @@
     <link name="base_link">
         <visual>
+            <origin xyz="0 0 ${baselen/2+0.05}" />
             <geometry>
                 <cylinder length="${baselen}" radius="0.2" />
@@ -37,5 +38,5 @@
         <parent link="base_link" />
         <child link="upper_base_link" />
-        <origin xyz="0 0 ${baselen/2+bodylen/2}" />
+        <origin xyz="0 0 ${(baselen+0.05)+bodylen/2}" />
     </joint>
     <!-- NECK -->
@@ -157,5 +158,5 @@
         <parent link="base_link" />
         <child link="ir_link" />
-        <origin xyz="0 0.2 0.3" rpy="0 0 0" />
+        <origin xyz="0 0.2 ${baselen/2+0.05+0.3}" rpy="0 0 0" />
     </joint>
     <!-- LASERS -->
@@ -166,5 +167,5 @@
         <parent link="base_link" />
         <child link="sick_link" />
-        <origin xyz="0 0.2 0" rpy="0 0 ${pi/2}" />
+        <origin xyz="0 0.2 ${baselen/2+0.05}" rpy="0 0 ${pi/2}" />
     </joint>
     <link name="hokuyo_link">
@@ -174,5 +175,5 @@
         <parent link="base_link" />
         <child link="hokuyo_link" />
-        <origin xyz="0 -0.2 0.2" rpy="0 0 -${pi/2}" />
+        <origin xyz="0 -0.2 ${baselen/2+0.05+0.2}" rpy="0 0 -${pi/2}" />
     </joint>
     <!-- TOUCH SENSORS -->
@@ -213,5 +214,5 @@
         <parent link="base_link" />
         <child link="kinect_link" />
-        <origin xyz="0 ${baselen/2+0.05} ${baselen/2+0.02}" rpy="0 0 0" />
+        <origin xyz="0 ${baselen/2+0.05} ${baselen+0.05+0.02}" rpy="0 0 0" />
     </joint>
     <link name="webcam_link">

File: maggie_description/urdf/wheels.urdf.xacro (robot description, xacro)
@@ -20,5 +20,5 @@
             <parent link="base_link" />
             <child link="${prefix}_wheel_link" />
-            <origin xyz="${reflect*0.1} 0 -0.18" rpy="0 0 0" />
+            <origin xyz="${reflect*0.1} 0 0.08" rpy="0 0 0" />
             <axis xyz="1 0 0" rpy="0 0 0" />
         </joint>
