Commit message: updated urdf

File: maggie_description/robots/maggie.urdf (robot description, URDF)
Before this commit: robot maggie, 26 links, 25 joints
Joints:
- joint base_to_hokuyo_joint: origin xyz=0 -0.2 0.46 rpy=0 0 -1.57075 -> xyz=0 -0.2 0.46 rpy=0 0 -3.1415
- joint base_to_sick_joint: origin xyz=0 0.2 0.26 rpy=0 0 1.57075 -> xyz=0 0.2 0.26 rpy=0 0 0

File: maggie_description/robots/maggie.urdf.xacro (robot description, xacro)
@@ -167,5 +167,5 @@
         <parent link="base_link" />
         <child link="sick_link" />
-        <origin xyz="0 0.2 ${baselen/2+0.05}" rpy="0 0 ${pi/2}" />
+        <origin xyz="0 0.2 ${baselen/2+0.05}" rpy="0 0 0" />
     </joint>
     <link name="hokuyo_link">
@@ -175,5 +175,5 @@
         <parent link="base_link" />
         <child link="hokuyo_link" />
-        <origin xyz="0 -0.2 ${baselen/2+0.05+0.2}" rpy="0 0 -${pi/2}" />
+        <origin xyz="0 -0.2 ${baselen/2+0.05+0.2}" rpy="0 0 -${pi}" />
     </joint>
     <!-- TOUCH SENSORS -->

Commit message: fixed wheels

File: maggie_description/robots/maggie.urdf (robot description, URDF)
Before this commit: robot maggie, 26 links, 25 joints
Links:
- removed link link_virtual
- added link virtual_link
Joints:
- joint base_to_left_wheel_joint: origin xyz=-0.1 0 0.08 rpy=0 0 0 -> xyz=0 -0.1 0.08 rpy=0 0 0
- joint base_to_right_wheel_joint: origin xyz=0.1 0 0.08 rpy=0 0 0 -> xyz=0 0.1 0.08 rpy=0 0 0
- joint base_to_tilt_head_joint: parent link_virtual -> virtual_link
- joint neck_to_pan_head_joint: child link_virtual -> virtual_link

File: maggie_description/robots/maggie.urdf.xacro (robot description, xacro)
@@ -61,8 +61,8 @@
     </joint>
     <!-- HEAD -->
-    <link name="link_virtual" />
+    <link name="virtual_link" />
     <joint name="neck_to_pan_head_joint" type="revolute">
         <parent link="neck_link" />
-        <child link="link_virtual" />
+        <child link="virtual_link" />
         <origin xyz="0 0 ${headlen/2}" />
         <axis xyz="0 0 1" />
@@ -84,5 +84,5 @@
     </link>
     <joint name="base_to_tilt_head_joint" type="revolute">
-        <parent link="link_virtual" />
+        <parent link="virtual_link" />
         <child link="head_link" />
         <origin xyz="0 0 0" />

File: maggie_description/urdf/wheels.urdf.xacro (robot description, xacro)
@@ -4,5 +4,5 @@
         <link name="${prefix}_wheel_link">
             <visual>
-                <origin xyz="0 0 0" rpy="0 0 ${pi/2}" />
+                <origin xyz="0 0 0" rpy="0 0 0" />
                 <geometry>
                     <mesh filename="package://maggie_description/meshes/base/wheel.dae" />
@@ -10,5 +10,5 @@
             </visual>
             <collision>
-                <origin xyz="0 0 0" rpy="0 0 ${pi/2}" />
+                <origin xyz="0 0 0" rpy="0 0 0" />
                 <geometry>
                     <mesh filename="package://maggie_description/meshes/base/wheel.dae" />
@@ -20,5 +20,5 @@
             <parent link="base_link" />
             <child link="${prefix}_wheel_link" />
-            <origin xyz="${reflect*0.1} 0 0.08" rpy="0 0 0" />
+            <origin xyz="0 ${reflect*0.1} 0.08" rpy="0 0 0" />
             <axis xyz="1 0 0" rpy="0 0 0" />
         </joint>

Commit message: fixed arms

File: maggie_description/robots/maggie.urdf (robot description, URDF)
Before this commit: robot maggie, 26 links, 25 joints
Joints:
- joint base_to_left_arm_joint: origin xyz=-0.25 0 0.28 -> xyz=0 -0.25 0.28
- joint base_to_right_arm_joint: origin xyz=0.25 0 0.28 -> xyz=0 0.25 0.28

File: maggie_description/urdf/arms.urdf.xacro (robot description, xacro)
@@ -4,5 +4,5 @@
         <link name="${prefix}_arm_link">
             <visual>
-                <origin xyz="0 0 ${-armlen/2}" rpy="0 ${pi/2} 0" />
+                <origin xyz="0 0 ${-armlen/2}" rpy="0 ${pi/2} ${pi/2}" />
                 <geometry>
                     <box size="${armlen} 0.15 0.1" />
@@ -21,5 +21,5 @@
             <parent link="upper_base_link" />
             <child link="${prefix}_arm_link" />
-            <origin xyz="${reflect*0.25} 0 ${bodylen/2}" />
+            <origin xyz="0 ${reflect*0.25} ${bodylen/2}" />
             <axis xyz="1 0 0" />
             <limit effort="1000.0" lower="-${pi/3}" upper="${3*pi/4}" velocity="${defaultvel}" />

Commit message: fixed eyes

File: maggie_description/robots/maggie.urdf (robot description, URDF)
Before this commit: robot maggie, 26 links, 25 joints
Joints:
- joint head_to_left_eye_joint: origin xyz=-0.06 0.16 0.05 -> xyz=0.16 -0.06 0.05
- joint head_to_right_eye_joint: origin xyz=0.06 0.16 0.05 -> xyz=0.16 0.06 0.05

File: maggie_description/urdf/eyes.urdf.xacro (robot description, xacro)
@@ -19,5 +19,5 @@
             <parent link="head_link" />
             <child link="${prefix}_eye_link" />
-            <origin xyz="${reflect*0.06} 0.16 0.05" />
+            <origin xyz="0.16 ${reflect*0.06} 0.05" />
         </joint>
     </xacro:macro>

Commit message: fixed mouth

File: maggie_description/robots/maggie.urdf (robot description, URDF)
Before this commit: robot maggie, 26 links, 25 joints
Joints:
- joint head_to_mouth_joint: origin xyz=0 0.17 -0.1 -> xyz=0.17 0 -0.1

File: maggie_description/robots/maggie.urdf.xacro (robot description, xacro)
@@ -93,4 +93,5 @@
     <link name="mouth_link">
         <visual>
+            <origin xyz="0 0 0" rpy="0 0 ${pi/2}" />
             <geometry>
                 <box size="0.1 0.02 0.02" />
@@ -108,5 +109,5 @@
         <parent link="head_link" />
         <child link="mouth_link" />
-        <origin xyz="0 0.17 -0.1" />
+        <origin xyz="0.17 0 -0.1" />
     </joint>
     <!-- EYES -->

Commit message: fixed screen

File: maggie_description/robots/maggie.urdf (robot description, URDF)
Before this commit: robot maggie, 26 links, 25 joints
Joints:
- joint base_to_screen_joint: origin xyz=0 0.19 0.105 -> xyz=0.19 0 0.105

File: maggie_description/robots/maggie.urdf.xacro (robot description, xacro)
@@ -122,4 +122,5 @@
     <link name="screen_link">
         <visual>
+            <origin xyz="0 0 0" rpy="0 0 ${pi/2}" />
             <geometry>
                 <box size="0.16 0.02 0.21" />
@@ -137,5 +138,5 @@
         <parent link="upper_base_link" />
         <child link="screen_link" />
-        <origin xyz="0 0.19 ${0.21/2}" />
+        <origin xyz="0.19 0 ${0.21/2}" />
     </joint>
     <!-- WHEELS -->

Commit message: fixed cameras

File: maggie_description/robots/maggie.urdf (robot description, URDF)
Before this commit: robot maggie, 26 links, 25 joints
Joints:
- joint base_to_kinect_joint: origin xyz=0 0.26 0.49 rpy=0 0 0 -> xyz=0.26 0 0.49 rpy=0 0 0

File: maggie_description/robots/maggie.urdf.xacro (robot description, xacro)
@@ -200,5 +200,5 @@
     <link name="kinect_link">
         <visual>
-            <origin xyz="0 0 0" rpy="0 0 ${pi/2}" />
+            <origin xyz="0 0 0" rpy="0 0 0" />
             <geometry>
                 <mesh filename="package://maggie_description/meshes/kinect/kinect.dae" scale="0.001 0.001 0.001" />
@@ -206,5 +206,5 @@
         </visual>
         <collision>
-            <origin xyz="0 0 0" rpy="0 0 ${pi/2}" />
+            <origin xyz="0 0 0" rpy="0 0 0" />
             <geometry>
                 <mesh filename="package://maggie_description/meshes/kinect/kinect.dae" scale="0.001 0.001 0.001" />
@@ -216,5 +216,5 @@
         <parent link="base_link" />
         <child link="kinect_link" />
-        <origin xyz="0 ${baselen/2+0.05} ${baselen+0.05+0.02}" rpy="0 0 0" />
+        <origin xyz="${baselen/2+0.05} 0 ${baselen+0.05+0.02}" rpy="0 0 0" />
     </joint>
     <link name="webcam_link">

Commit message: fixed lasers

File: maggie_description/robots/maggie.urdf (robot description, URDF)
Before this commit: robot maggie, 26 links, 25 joints
Joints:
- joint base_to_hokuyo_joint: origin xyz=0 -0.2 0.46 rpy=0 0 -3.1415 -> xyz=-0.2 0 0.46 rpy=0 0 -3.1415
- joint base_to_sick_joint: origin xyz=0 0.2 0.26 rpy=0 0 0 -> xyz=0.2 0 0.26 rpy=0 0 0

File: maggie_description/robots/maggie.urdf.xacro (robot description, xacro)
@@ -169,5 +169,5 @@
         <parent link="base_link" />
         <child link="sick_link" />
-        <origin xyz="0 0.2 ${baselen/2+0.05}" rpy="0 0 0" />
+        <origin xyz="0.2 0 ${baselen/2+0.05}" rpy="0 0 0" />
     </joint>
     <link name="hokuyo_link">
@@ -177,5 +177,5 @@
         <parent link="base_link" />
         <child link="hokuyo_link" />
-        <origin xyz="0 -0.2 ${baselen/2+0.05+0.2}" rpy="0 0 -${pi}" />
+        <origin xyz="-0.2 0 ${baselen/2+0.05+0.2}" rpy="0 0 -${pi}" />
     </joint>
     <!-- TOUCH SENSORS -->

Commit message: fixed ir and rfid

File: maggie_description/robots/maggie.urdf (robot description, URDF)
Before this commit: robot maggie, 26 links, 25 joints
Joints:
- joint base_to_ir_joint: origin xyz=0 0.2 0.56 rpy=0 0 0 -> xyz=0.2 0 0.56 rpy=0 0 0
- joint head_to_rfid_joint: origin xyz=0 0.2 0 rpy=0 0 0 -> xyz=0.2 0 0 rpy=0 0 0

File: maggie_description/robots/maggie.urdf.xacro (robot description, xacro)
@@ -151,5 +151,5 @@
         <parent link="head_link" />
         <child link="rfid_link" />
-        <origin xyz="0 0.2 0" rpy="0 0 0" />
+        <origin xyz="0.2 0 0" rpy="0 0 0" />
     </joint>
     <!-- IR CONTROLLER -->
@@ -160,5 +160,5 @@
         <parent link="base_link" />
         <child link="ir_link" />
-        <origin xyz="0 0.2 ${baselen/2+0.05+0.3}" rpy="0 0 0" />
+        <origin xyz="0.2 0 ${baselen/2+0.05+0.3}" rpy="0 0 0" />
     </joint>
     <!-- LASERS -->

Commit message: fixed moves

File: maggie_description/robots/maggie.urdf (robot description, URDF)
Before this commit: robot maggie, 26 links, 25 joints
Joints:
- joint base_to_left_arm_joint: axis 1 0 0 -> 0 1 0
- joint base_to_left_wheel_joint: axis 1 0 0 -> 0 1 0
- joint base_to_right_arm_joint: axis 1 0 0 -> 0 1 0
- joint base_to_right_wheel_joint: axis 1 0 0 -> 0 1 0
- joint base_to_tilt_head_joint: axis 1 0 0 -> 0 1 0

File: maggie_description/robots/maggie.urdf.xacro (robot description, xacro)
@@ -87,5 +87,5 @@
         <child link="head_link" />
         <origin xyz="0 0 0" />
-        <axis xyz="1 0 0" />
+        <axis xyz="0 1 0" />
         <limit effort="1000.0" lower="-0.26" upper="0.26" velocity="${defaultvel}" />
     </joint>

File: maggie_description/urdf/arms.urdf.xacro (robot description, xacro)
@@ -22,5 +22,5 @@
             <child link="${prefix}_arm_link" />
             <origin xyz="0 ${reflect*0.25} ${bodylen/2}" />
-            <axis xyz="1 0 0" />
+            <axis xyz="0 1 0" />
             <limit effort="1000.0" lower="-${pi/3}" upper="${3*pi/4}" velocity="${defaultvel}" />
         </joint>

File: maggie_description/urdf/wheels.urdf.xacro (robot description, xacro)
@@ -21,5 +21,5 @@
             <child link="${prefix}_wheel_link" />
             <origin xyz="0 ${reflect*0.1} 0.08" rpy="0 0 0" />
-            <axis xyz="1 0 0" rpy="0 0 0" />
+            <axis xyz="0 1 0" rpy="0 0 0" />
         </joint>
     </xacro:macro>
